Commit message: sistemato

File: urdf/my_robot_x.urdf (robot description, URDF)
Before this commit: robot my_robot, 5 links, 4 joints
Links:
- link base_link: mass None -> 5

File: urdf/my_robot_x.xacro (robot description, xacro)
@@ -31,4 +31,8 @@
       </geometry>
     </collision>
+      <inertial>
+        <mass value="${base_mass}" />
+        <cylinder_inertia m="${base_mass}" r="${base_radius}" h="${base_height}"/>
+      </inertial>
   </link>
 <!--
