Commit message: modifiche

File: urdf/my_robot_x.xacro (robot description, xacro)
@@ -1,5 +1,6 @@
 <?xml version="1.0"?>
 <robot name="my_robot" xmlns:xacro="http://www.ros.org/wiki/xacro">
-  <xacro:include filename="$(find my_robot_urdf)/urdf/cylinder_wheel.urdf.xacro"/>
+  <xacro:include filename="$(find ackermann)/urdf/cylinder_wheel.urdf.xacro"/>
+  <xacro:include filename="$(find ackermann)/urdf/sterzanti.xacro"/>
   <!--<xacro:include filename="$(find my_robot_urdf)/urdf/caster_wheel.urdf.xacro"/>-->
   <!--PROPERTY LIST-->
@@ -9,5 +10,5 @@
   <xacro:property name="DEG_TO_RAD" value="0.017453293"/>
   <!--Main Body cylinder base -->
-  <xacro:property name="base_height" value="0.02"/>
+  <xacro:property name="base_height" value="0.2"/>
   <xacro:property name="base_radius" value="0.15"/>
   <xacro:property name="base_mass" value="5"/> <!-- in kg -->
@@ -19,5 +20,5 @@
     <visual>
       <geometry>
-      <box size="0.5 0.25 0.125" />
+      <box size="0.25 0.110 0.03" />
       <!--<cylinder length="${base_height}" radius="0.15"/>-->
       </geometry>
@@ -27,5 +28,5 @@
     <collision>
       <geometry>
-      <box size="0.5 0.25 0.125" />
+      <box size="0.25 0.110 0.03" />
       <!--<cylinder radius="${base_radius}" length="${base_height}"/>-->
       </geometry>
@@ -36,12 +37,8 @@
       </inertial>
   </link>
-<!--
-  <caster_wheel fb="caster" lr="front" assex="0" parent="base_link" originx="0.115" originz="0.007"/>
-  <caster_wheel fb="caster" lr="back" assex="0.02" parent="base_link" originx="-0.135" originz="0.009"/>
--->
-  <cylinder_wheel fb="front" lr="right" parent="base_link" translateX="-1" translateY="0.42" flipY="1"/>
-  <cylinder_wheel fb="front" lr="left" parent="base_link" translateX="-1" translateY="-0.42" flipY="1"/>
-  <cylinder_wheel fb="rear" lr="right" parent="base_link" translateX="1" translateY="0.42" flipY="1"/>
-  <cylinder_wheel fb="rear" lr="left" parent="base_link" translateX="1" translateY="-0.42" flipY="1"/>
+  <cylinder_wheel fb="rear" lr="right" parent="base_link" translateX="-0.5" translateY="0.212" flipY="1"/>
+  <cylinder_wheel fb="rear" lr="left" parent="base_link" translateX="-0.5" translateY="-0.212" flipY="1"/>
+  <cylinder_steering_wheel fb="front" lr="right" parent="base_link" translateX="0.5" translateY="0.212" flipY="1"/>
+  <cylinder_steering_wheel fb="front" lr="left" parent="base_link" translateX="0.5" translateY="-0.212" flipY="1"/>
   <gazebo>
     <plugin name="gazebo_ros_control" filename="libgazebo_ros_control.so">

File: urdf/sterzanti.xacro (robot description, xacro)
@@ -13,5 +13,5 @@
               izz="${m*r*r/2}" />
   </xacro:macro>
-  <xacro:macro name="cylinder_wheel" params="fb lr parent translateX translateY flipY"> <!--fb : front, back ; lr: left, right -->
+  <xacro:macro name="cylinder_steering_wheel" params="fb lr parent translateX translateY flipY"> <!--fb : front, back ; lr: left, right -->
     <link name="${fb}_${lr}_wheel">
       <visual>
@@ -43,5 +43,5 @@
       <turnGravityOff>false</turnGravityOff>
     </gazebo>
-    <joint name="${fb}_${lr}_wheel_joint" type="continuous">
+    <joint name="${fb}_${lr}_wheel_joint" type="revolute">
       <parent link="${parent}"/>
       <child link="${fb}_${lr}_wheel"/>
@@ -51,5 +51,5 @@
       <joint_properties damping="0.0" friction="0.0"/>
     </joint>
-    <!-- Transmission is important to link the joints and the controller -->
+     <!-- Transmission is important to link the joints and the controller -->
     <transmission name="${fb}_${lr}_wheel_joint_trans">
       <type>transmission_interface/SimpleTransmission</type>
