Commit message: modifiche

File: urdf/cylinder_wheel.urdf.xacro (robot description, xacro)
@@ -5,6 +5,8 @@
   <xacro:property name="wheel_height" value="0.02" />
   <xacro:property name="wheel_mass" value="2.5" /> <!-- in kg-->
+  <!--
   <xacro:property name="base_x_origin_to_wheel_origin" value="0.25" />
   <xacro:property name="base_y_origin_to_wheel_origin" value="0.3" />
+    -->
   <xacro:property name="base_z_origin_to_wheel_origin" value="0.0" />
   <xacro:macro name="cylinder_inertia" params="m r h">
@@ -46,5 +48,8 @@
       <parent link="${parent}"/>
       <child link="${fb}_${lr}_wheel"/>
+      <origin xyz="${translateX} ${translateY} ${base_z_origin_to_wheel_origin}" rpy="0 0 0" />
+      <!--
       <origin xyz="${translateX * base_x_origin_to_wheel_origin} ${translateY * base_y_origin_to_wheel_origin} ${base_z_origin_to_wheel_origin}" rpy="0 0 0" />
+      -->
       <axis xyz="0 1 0" rpy="0  0" />
       <limit effort="100" velocity="100"/>

File: urdf/my_robot_x.xacro (robot description, xacro)
@@ -2,10 +2,18 @@
 <robot name="my_robot" xmlns:xacro="http://www.ros.org/wiki/xacro">
   <xacro:include filename="$(find my_robot_urdf)/urdf/cylinder_wheel.urdf.xacro"/>
-  <xacro:include filename="$(find my_robot_urdf)/urdf/caster_wheel.urdf.xacro"/>
-  <xacro:include filename="$(find my_robot_urdf)/urdf/visual_sensor.xacro"/>
+  <!--PROPERTY LIST-->
+  <!--All units in m-kg-s-radians unit system -->
+  <xacro:property name="M_PI" value="3.1415926535897931"/>
+  <xacro:property name="M_PI_2" value="1.570796327"/>
+  <xacro:property name="DEG_TO_RAD" value="0.017453293"/>
+  <!--Main Body cylinder base -->
+  <xacro:property name="base_height" value="0.02"/>
+  <xacro:property name="base_radius" value="0.15"/>
+  <xacro:property name="base_mass" value="5"/> <!-- in kg -->
   <link name="base_link">
     <visual>
       <geometry>
-        <cylinder length="${base_height}" radius="0.15"/>
+       <box size="0.5 0.25 0.115" />
+       <!-- <cylinder length="${base_height}" radius="0.15"/>-->
       </geometry>
       <origin rpy="0 0 0" xyz="0 0 0"/>
@@ -14,12 +22,11 @@
     <collision>
       <geometry>
-        <cylinder radius="${base_radius}" length="${base_height}"/>
+      <box size="0.5 0.25 0.115" />
+      <!--<cylinder radius="${base_radius}" length="${base_height}"/>-->
       </geometry>
     </collision>
   </link>
-  <caster_wheel fb="caster" lr="front" assex="0" parent="base_link" originx="0.115" originz="0.007"/>
-  <caster_wheel fb="caster" lr="back" assex="0.02" parent="base_link" originx="-0.135" originz="0.009"/>
-  <cylinder_wheel fb="front" lr="right" parent="base_link" translateX="0" translateY="0.5" flipY="1"/>
-  <cylinder_wheel fb="front" lr="left" parent="base_link" translateX="0" translateY="-0.5" flipY="1"/>
+  <cylinder_wheel fb="front" lr="right" parent="base_link" translateX="0.25" translateY="0.115" flipY="1"/>
+  <cylinder_wheel fb="front" lr="left" parent="base_link" translateX="0.25" translateY="-0.115" flipY="1"/>
   <hokuyo base_radius="${base_radius}" base_height="${base_height}"/>
   <gazebo>

Commit message: modifiche

File: urdf/cylinder_wheel.urdf.xacro (robot description, xacro)
@@ -2,11 +2,9 @@
 <robot name="my_robot" xmlns:xacro="http://www.ros.org/wiki/xacro">
   <!-- Wheels -->
-  <xacro:property name="wheel_radius" value="0.04" />
+  <xacro:property name="wheel_radius" value="0.4" />
   <xacro:property name="wheel_height" value="0.02" />
   <xacro:property name="wheel_mass" value="2.5" /> <!-- in kg-->
-  <!--
   <xacro:property name="base_x_origin_to_wheel_origin" value="0.25" />
   <xacro:property name="base_y_origin_to_wheel_origin" value="0.3" />
-    -->
   <xacro:property name="base_z_origin_to_wheel_origin" value="0.0" />
   <xacro:macro name="cylinder_inertia" params="m r h">
@@ -48,8 +46,5 @@
       <parent link="${parent}"/>
       <child link="${fb}_${lr}_wheel"/>
-      <origin xyz="${translateX} ${translateY} ${base_z_origin_to_wheel_origin}" rpy="0 0 0" />
-      <!--
       <origin xyz="${translateX * base_x_origin_to_wheel_origin} ${translateY * base_y_origin_to_wheel_origin} ${base_z_origin_to_wheel_origin}" rpy="0 0 0" />
-      -->
       <axis xyz="0 1 0" rpy="0  0" />
       <limit effort="100" velocity="100"/>

File: urdf/my_robot_x.urdf (robot description, URDF)
Before this commit: robot my_robot, 3 links, 2 joints
Links:
- added link rear_left_wheel, mass 2.5; collision cylinder length=0.02 radius=0.04; visual cylinder length=0.02 radius=0.04
- added link rear_right_wheel, mass 2.5; collision cylinder length=0.02 radius=0.04; visual cylinder length=0.02 radius=0.04
- link base_link: geometry collision box size=0.5 0.25 0.125; visual box size=0.5 0.25 0.125
Joints:
- added joint rear_left_wheel_joint: type continuous, parent base_link, child rear_left_wheel, origin xyz=0.25 -0.126 0.0 rpy=0 0 0, axis 0 1 0, limit effort=100 velocity=100
- added joint rear_right_wheel_joint: type continuous, parent base_link, child rear_right_wheel, origin xyz=0.25 0.126 0.0 rpy=0 0 0, axis 0 1 0, limit effort=100 velocity=100
- joint front_left_wheel_joint: origin xyz=0.0 -0.045 0.0 rpy=0 0 0 -> xyz=-0.25 -0.126 0.0 rpy=0 0 0
- joint front_right_wheel_joint: origin xyz=0.0 0.045 0.0 rpy=0 0 0 -> xyz=-0.25 0.126 0.0 rpy=0 0 0

File: urdf/my_robot_x.xacro (robot description, xacro)
@@ -2,4 +2,5 @@
 <robot name="my_robot" xmlns:xacro="http://www.ros.org/wiki/xacro">
   <xacro:include filename="$(find my_robot_urdf)/urdf/cylinder_wheel.urdf.xacro"/>
+  <!--<xacro:include filename="$(find my_robot_urdf)/urdf/caster_wheel.urdf.xacro"/>-->
   <!--PROPERTY LIST-->
   <!--All units in m-kg-s-radians unit system -->
@@ -11,9 +12,13 @@
   <xacro:property name="base_radius" value="0.15"/>
   <xacro:property name="base_mass" value="5"/> <!-- in kg -->
+  <!-- Caster wheel -->
+  <xacro:property name="caster_height" value="0.04"/>
+  <xacro:property name="caster_radius" value="0.025"/>
+  <xacro:property name="caster_mass" value="0.5"/>
   <link name="base_link">
     <visual>
       <geometry>
-       <box size="0.5 0.25 0.115" />
-       <!-- <cylinder length="${base_height}" radius="0.15"/>-->
+      <box size="0.5 0.25 0.125" />
+      <!--<cylinder length="${base_height}" radius="0.15"/>-->
       </geometry>
       <origin rpy="0 0 0" xyz="0 0 0"/>
@@ -22,12 +27,17 @@
     <collision>
       <geometry>
-      <box size="0.5 0.25 0.115" />
+      <box size="0.5 0.25 0.125" />
       <!--<cylinder radius="${base_radius}" length="${base_height}"/>-->
       </geometry>
     </collision>
   </link>
-  <cylinder_wheel fb="front" lr="right" parent="base_link" translateX="0.25" translateY="0.115" flipY="1"/>
-  <cylinder_wheel fb="front" lr="left" parent="base_link" translateX="0.25" translateY="-0.115" flipY="1"/>
-  <hokuyo base_radius="${base_radius}" base_height="${base_height}"/>
+<!--
+  <caster_wheel fb="caster" lr="front" assex="0" parent="base_link" originx="0.115" originz="0.007"/>
+  <caster_wheel fb="caster" lr="back" assex="0.02" parent="base_link" originx="-0.135" originz="0.009"/>
+-->
+  <cylinder_wheel fb="front" lr="right" parent="base_link" translateX="-1" translateY="0.42" flipY="1"/>
+  <cylinder_wheel fb="front" lr="left" parent="base_link" translateX="-1" translateY="-0.42" flipY="1"/>
+  <cylinder_wheel fb="rear" lr="right" parent="base_link" translateX="1" translateY="0.42" flipY="1"/>
+  <cylinder_wheel fb="rear" lr="left" parent="base_link" translateX="1" translateY="-0.42" flipY="1"/>
   <gazebo>
     <plugin name="gazebo_ros_control" filename="libgazebo_ros_control.so">

Commit message: progetto ripristinato

File: urdf/cylinder_wheel.urdf.xacro (robot description, xacro)
@@ -1,4 +1,4 @@
 <?xml version="1.0"?>
-<robot name="my_robot" xmlns:xacro="http://www.ros.org/wiki/xacro">
+<robot name="ackermann" xmlns:xacro="http://www.ros.org/wiki/xacro">
   <!-- Wheels -->
   <xacro:property name="wheel_radius" value="0.04" />

File: urdf/sterzanti.xacro (robot description, xacro)
@@ -1,4 +1,4 @@
 <?xml version="1.0"?>
-<robot name="my_robot" xmlns:xacro="http://www.ros.org/wiki/xacro">
+<robot name="ackermann" xmlns:xacro="http://www.ros.org/wiki/xacro">
   <!-- Wheels -->
   <xacro:property name="wheel_radius" value="0.04" />
@@ -51,14 +51,14 @@
       <joint_properties damping="0.0" friction="0.0"/>
     </joint>
-     <!-- Transmission is important to link the joints and the controller -->
     <transmission name="${fb}_${lr}_wheel_joint_trans">
-      <type>transmission_interface/SimpleTransmission</type>
-      <joint name="${fb}_${lr}_wheel_joint">
-        <hardwareInterface>hardware_interface/VelocityJointInterface</hardwareInterface>
-      </joint>
-      <actuator name="${fb}_${lr}_wheel_joint_motor">
-        <mechanicalReduction>1</mechanicalReduction>
-      </actuator>
-    </transmission>
+    <type>transmission_interface/SimpleTransmission</type>
+    <joint name="${fb}_${lr}_wheel_joint">
+    <hardwareInterface>EffortJointInterface</hardwareInterface>
+    </joint>
+    <actuator name="${fb}_${lr}_wheel_joint_motor">
+      <hardwareInterface>EffortJointInterface</hardwareInterface>
+      <mechanicalReduction>1</mechanicalReduction>
+    </actuator>
+  </transmission>
   </xacro:macro>
 </robot>
