Commit message: fari

File: urdf/car.xacro (robot description, xacro)
@@ -3,4 +3,5 @@
   <xacro:include filename="$(find ackermann)/urdf/cylinder_wheel.urdf.xacro"/>
   <xacro:include filename="$(find ackermann)/urdf/sterzanti.xacro"/>
+  <xacro:include filename="$(find ackermann)/urdf/fari.xacro"/>
   <!--PROPERTY LIST-->
   <!--All units in m-kg-s-radians unit system -->
@@ -8,17 +9,12 @@
   <xacro:property name="M_PI_2" value="1.570796327"/>
   <xacro:property name="DEG_TO_RAD" value="0.017453293"/>
-  <!--Main Body cylinder base -->
+  <!--Main Body box base -->
   <xacro:property name="base_height" value="0.2"/>
   <xacro:property name="base_radius" value="0.15"/>
   <xacro:property name="base_mass" value="5"/> <!-- in kg -->
-  <!-- Caster wheel -->
-  <xacro:property name="caster_height" value="0.04"/>
-  <xacro:property name="caster_radius" value="0.025"/>
-  <xacro:property name="caster_mass" value="0.5"/>
   <link name="base_link">
     <visual>
       <geometry>
-      <box size="0.25 0.110 0.03" />
-      <!--<cylinder length="${base_height}" radius="0.15"/>-->
+      <box size="0.25 0.110 0.01" />
       </geometry>
       <origin rpy="0 0 0" xyz="0 0 0"/>
@@ -27,5 +23,5 @@
     <collision>
       <geometry>
-      <box size="0.25 0.110 0.03" />
+      <box size="0.25 0.110 0.01" />
       <!--<cylinder radius="${base_radius}" length="${base_height}"/>-->
       </geometry>
@@ -36,8 +32,10 @@
       </inertial>
   </link>
-  <cylinder_wheel fb="rear" lr="right" parent="base_link" translateX="-0.5" translateY="0.212" flipY="1"/>
-  <cylinder_wheel fb="rear" lr="left" parent="base_link" translateX="-0.5" translateY="-0.212" flipY="1"/>
-  <cylinder_steering_wheel fb="front" lr="right" parent="base_link" translateX="0.5" translateY="0.212" flipY="1"/>
-  <cylinder_steering_wheel fb="front" lr="left" parent="base_link" translateX="0.5" translateY="-0.212" flipY="1"/>
+  <cylinder_wheel fb="rear" lr="right" parent="base_link" translateX="-0.5" translateY="0.272" flipY="1"/>
+  <cylinder_wheel fb="rear" lr="left" parent="base_link" translateX="-0.5" translateY="-0.272" flipY="1"/>
+  <cylinder_steering_wheel fb="front" lr="right" parent="base_link" translateX="0.5" translateY="0.272" flipY="1"/>
+  <cylinder_steering_wheel fb="front" lr="left" parent="base_link" translateX="0.5" translateY="-0.272" flipY="1"/>
+  <faro fb ="front" lr="right" parent="base_link" translateX="0.45" translateY="0.1" flipY="1" />
+  <faro fb ="front" lr="left" parent="base_link" translateX="0.45" translateY="-0.1" flipY="1" />
   <gazebo>
     <plugin name="gazebo_ros_control" filename="libgazebo_ros_control.so">

File: urdf/cylinder_wheel.urdf.xacro (robot description, xacro)
@@ -3,5 +3,5 @@
   <!-- Wheels -->
   <xacro:property name="wheel_radius" value="0.04" />
-  <xacro:property name="wheel_height" value="0.02" />
+  <xacro:property name="wheel_height" value="0.04" />
   <xacro:property name="wheel_mass" value="2.5" /> <!-- in kg-->
   <xacro:property name="base_x_origin_to_wheel_origin" value="0.25" />

File: urdf/sterzanti.xacro (robot description, xacro)
@@ -3,5 +3,5 @@
   <!-- Wheels -->
   <xacro:property name="wheel_radius" value="0.04" />
-  <xacro:property name="wheel_height" value="0.02" />
+  <xacro:property name="wheel_height" value="0.04" />
   <xacro:property name="wheel_mass" value="2.5" /> <!-- in kg-->
   <xacro:property name="base_x_origin_to_wheel_origin" value="0.25" />

Commit message: inerzia corretta

File: urdf/car.xacro (robot description, xacro)
@@ -9,12 +9,20 @@
   <xacro:property name="M_PI_2" value="1.570796327"/>
   <xacro:property name="DEG_TO_RAD" value="0.017453293"/>
-  <!--Main Body box base -->
-  <xacro:property name="base_height" value="0.2"/>
-  <xacro:property name="base_radius" value="0.15"/>
-  <xacro:property name="base_mass" value="5"/> <!-- in kg -->
+  <!--Main Body box base  (z y x)-->
+  <xacro:property name="height" value="0.01"/>
+  <xacro:property name="width" value="0.110"/>
+  <xacro:property name="depth" value="0.25"/>
+  <xacro:property name="mass" value="5"/> <!-- in kg -->
+  <xacro:macro name="solid_cuboid_inertial" params="width depth height mass">
+      <inertia ixx="${mass * (depth * depth + height * height) / 12}"
+               ixy="0" ixz="0"
+               iyy="${mass * (width * width + height * height) / 12}"
+               iyz="0"
+               izz="${mass * (width * width + depth * depth) / 12}"/>
+  </xacro:macro>
   <link name="base_link">
     <visual>
       <geometry>
-      <box size="0.25 0.110 0.01" />
+      <box size="${depth} ${width} ${height}"/>
       </geometry>
       <origin rpy="0 0 0" xyz="0 0 0"/>
@@ -24,10 +32,10 @@
       <geometry>
       <box size="0.25 0.110 0.01" />
-      <!--<cylinder radius="${base_radius}" length="${base_height}"/>-->
+      <!--<cylinder radius="${base_radius}" length="${height}"/>-->
       </geometry>
     </collision>
       <inertial>
-        <mass value="${base_mass}" />
-        <cylinder_inertia m="${base_mass}" r="${base_radius}" h="${base_height}"/>
+        <mass value="${mass}" />
+        <solid_cuboid_inertial width='${width}' depth='${depth}' height='${height}' mass='${mass}' />
       </inertial>
   </link>
