Commit message: sterzanti

File: urdf/sterzanti.xacro (robot description, xacro)
@@ -47,6 +47,6 @@
       <child link="${fb}_${lr}_wheel"/>
       <origin xyz="${translateX * base_x_origin_to_wheel_origin} ${translateY * base_y_origin_to_wheel_origin} ${base_z_origin_to_wheel_origin}" rpy="0 0 0" />
-      <axis xyz="0 1 0" rpy="0  0" />
-      <limit effort="100" velocity="100"/>
+      <axis xyz="0 0 1" rpy="0  0" />
+      <limit lower="-0.78" upper="0.78" effort="100" velocity="100"/>
       <joint_properties damping="0.0" friction="0.0"/>
     </joint>
@@ -57,5 +57,5 @@
     </joint>
     <actuator name="${fb}_${lr}_wheel_joint_motor">
-      <hardwareInterface>PositionJointInterface</hardwareInterface>
+      <hardwareInterface>EffortJointInterface</hardwareInterface>
       <mechanicalReduction>1</mechanicalReduction>
     </actuator>

Commit message: wasd_class inserito

File: urdf/sterzanti.xacro (robot description, xacro)
@@ -43,5 +43,5 @@
       <turnGravityOff>false</turnGravityOff>
     </gazebo>
-    <joint name="${fb}_${lr}_wheel_joint" type="revolute">
+    <joint name="${fb}_${lr}_wheel_joint" type="continuous">
       <parent link="${parent}"/>
       <child link="${fb}_${lr}_wheel"/>

Commit message: understanding slipping error

File: urdf/sterzanti.xacro (robot description, xacro)
@@ -47,9 +47,11 @@
       <child link="${fb}_${lr}_wheel"/>
       <origin xyz="${translateX * base_x_origin_to_wheel_origin} ${translateY * base_y_origin_to_wheel_origin} ${base_z_origin_to_wheel_origin}" rpy="0 0 0" />
-      <axis xyz="0 0 1" rpy="0  0" />
-      <limit lower="-0.78" upper="0.78" effort="100" velocity="100"/>
+      <axis xyz="0 1 0" rpy="0 0 0" />
+      <!--<axis xyz="0 0 1" rpy="0  0" />-->
+      <!--<limit lower="-0.78" upper="0.78" effort="100" velocity="100"/>-->
       <joint_properties damping="0.0" friction="0.0"/>
     </joint>
-    <transmission name="${fb}_${lr}_wheel_joint_trans">
+<!--
+  <transmission name="${fb}_${lr}_wheel_joint_trans">
     <type>transmission_interface/SimpleTransmission</type>
     <joint name="${fb}_${lr}_wheel_joint">
@@ -61,4 +63,5 @@
     </actuator>
   </transmission>
+-->
   </xacro:macro>
 </robot>
