Commit message: problema strisciamento

File: urdf/car.urdf (robot description, URDF)
Before this commit: robot ackermann, 5 links, 4 joints
Links:
- added link front_left_axle_carrier, mass 0.001
- added link front_left_light, mass 5; collision cylinder length=0.01 radius=0.015; visual cylinder length=0.01 radius=0.015
- added link front_right_axle_carrier, mass 0.001
- added link front_right_light, mass 5; collision cylinder length=0.01 radius=0.015; visual cylinder length=0.01 radius=0.015
- link base_link: geometry collision box size=0.25 0.110 0.01; visual box size=0.25 0.11 0.01
- link front_left_wheel: geometry collision cylinder length=0.04 radius=0.04; visual cylinder length=0.04 radius=0.04
- link front_right_wheel: geometry collision cylinder length=0.04 radius=0.04; visual cylinder length=0.04 radius=0.04
- link rear_left_wheel: geometry collision cylinder length=0.04 radius=0.04; visual cylinder length=0.04 radius=0.04
- link rear_right_wheel: geometry collision cylinder length=0.04 radius=0.04; visual cylinder length=0.04 radius=0.04
Joints:
- added joint front_left_light_joint: type fixed, parent base_link, child front_left_light, origin xyz=0.1125 -0.03 0.01 rpy=0 0 0, axis 0 1 0
- added joint front_left_steering_wheel_joint: type revolute, parent front_left_axle_carrier, child front_left_wheel, origin xyz=0.125 -0.0816 0.0 rpy=0 0 0, axis 0 0 1, limit lower=-0.78 upper=0.78 effort=100 velocity=100
- added joint front_right_light_joint: type fixed, parent base_link, child front_right_light, origin xyz=0.1125 0.03 0.01 rpy=0 0 0, axis 0 1 0
- added joint front_right_steering_wheel_joint: type revolute, parent front_right_axle_carrier, child front_right_wheel, origin xyz=0.125 0.0816 0.0 rpy=0 0 0, axis 0 0 1, limit lower=-0.78 upper=0.78 effort=100 velocity=100
- joint front_left_wheel_joint: axis 0 0 1 -> 0 1 0; child front_left_wheel -> front_left_axle_carrier; limit lower=-0.78 upper=0.78 effort=100 velocity=100 -> (none); origin xyz=0.125 -0.0636 0.0 rpy=0 0 0 -> xyz=0.125 -0.0816 0.0 rpy=0 0 0; type revolute -> continuous
- joint front_right_wheel_joint: axis 0 0 1 -> 0 1 0; child front_right_wheel -> front_right_axle_carrier; limit lower=-0.78 upper=0.78 effort=100 velocity=100 -> (none); origin xyz=0.125 0.0636 0.0 rpy=0 0 0 -> xyz=0.125 0.0816 0.0 rpy=0 0 0; type revolute -> continuous
- joint rear_left_wheel_joint: origin xyz=-0.125 -0.0636 0.0 rpy=0 0 0 -> xyz=-0.125 -0.0816 0.0 rpy=0 0 0
- joint rear_right_wheel_joint: origin xyz=-0.125 0.0636 0.0 rpy=0 0 0 -> xyz=-0.125 0.0816 0.0 rpy=0 0 0

File: urdf/car.xacro (robot description, xacro)
@@ -21,4 +21,12 @@
                izz="${mass * (width * width + depth * depth) / 12}"/>
   </xacro:macro>
+  <!--Rimozione warning
+  <link name="chasis">
+  </link>
+  <joint name="chasis_joint" type="fixed">
+  <parent link="chasis"/>
+  <child link="base_link"/>
+  </joint>
+-->
   <link name="base_link">
     <visual>
@@ -32,5 +40,4 @@
       <geometry>
       <box size="0.25 0.110 0.01" />
-      <!--<cylinder radius="${base_radius}" length="${height}"/>-->
       </geometry>
     </collision>

File: urdf/sterzanti.xacro (robot description, xacro)
@@ -13,5 +13,14 @@
               izz="${m*r*r/2}" />
   </xacro:macro>
+   <xacro:macro name="null_inertial">
+    <inertial>
+      <mass value="0.001"/>
+      <inertia ixx="0.001" ixy="0" ixz="0" iyy="0.001" iyz="0" izz="0.001"/>
+    </inertial>
+  </xacro:macro>
   <xacro:macro name="cylinder_steering_wheel" params="fb lr parent translateX translateY flipY"> <!--fb : front, back ; lr: left, right -->
+    <link name="${fb}_${lr}_axle_carrier">
+      <xacro:null_inertial/>
+    </link>
     <link name="${fb}_${lr}_wheel">
       <visual>
@@ -44,7 +53,7 @@
     </gazebo>
     <joint name="${fb}_${lr}_wheel_joint" type="continuous">
-      <parent link="${parent}"/>
+      <parent link="${fb}_${lr}_axle_carrier"/>
       <child link="${fb}_${lr}_wheel"/>
-      <origin xyz="${translateX * base_x_origin_to_wheel_origin} ${translateY * base_y_origin_to_wheel_origin} ${base_z_origin_to_wheel_origin}" rpy="0 0 0" />
+      <origin xyz="0 0 0" rpy="0 0 0"/>
       <axis xyz="0 1 0" rpy="0 0 0" />
       <!--<axis xyz="0 0 1" rpy="0  0" />-->
@@ -52,8 +61,15 @@
       <joint_properties damping="0.0" friction="0.0"/>
     </joint>
-<!--
+   <joint name="${fb}_${lr}_steering_wheel_joint" type="revolute">
+      <parent link="${parent}"/>
+      <child link="${fb}_${lr}_axle_carrier"/>
+      <origin xyz="${translateX * base_x_origin_to_wheel_origin} ${translateY * base_y_origin_to_wheel_origin} ${base_z_origin_to_wheel_origin}" rpy="0 0 0" />
+      <axis xyz="0 0 1" rpy="0 0 0" />
+      <limit lower="-0.78" upper="0.78" effort="100" velocity="100"/>
+      <joint_properties damping="0.0" friction="0.0"/>
+    </joint>
   <transmission name="${fb}_${lr}_wheel_joint_trans">
     <type>transmission_interface/SimpleTransmission</type>
-    <joint name="${fb}_${lr}_wheel_joint">
+    <joint name="${fb}_${lr}_steering_wheel_joint">
     <hardwareInterface>hardware_interface/PositionJointInterface</hardwareInterface>
     </joint>
@@ -63,5 +79,13 @@
     </actuator>
   </transmission>
--->
+  <transmission name="${fb}_${lr}_wheel_joint_trans1">
+      <type>transmission_interface/SimpleTransmission</type>
+      <joint name="${fb}_${lr}_wheel_joint">
+        <hardwareInterface>hardware_interface/VelocityJointInterface</hardwareInterface>
+      </joint>
+      <actuator name="${fb}_${lr}_wheel_joint_motor1">
+        <mechanicalReduction>1</mechanicalReduction>
+      </actuator>
+  </transmission>
   </xacro:macro>
 </robot>
